Commit message: Checkpoint

File: genRobot.urdf (robot description, URDF)
Before this commit: robot test_robot, 8 links, 7 joints
Links:
- removed link scanner
- link lwheel: mass None -> 0.1
- link rwheel: mass None -> 0.1
Joints:
- removed joint base_to_scanner
- joint base_to_lwheel: origin xyz=-0.05 0.115 0.046 rpy=0 0 1.5707963 -> xyz=-0.05 0.115 0.046 rpy=0 0 -1.5707963
- joint base_to_rwheel: origin xyz=-0.05 -0.115 0.046 rpy=0 0 -1.5707963 -> xyz=-0.05 -0.115 0.046 rpy=0 0 1.5707963

Commit message: Checkpoint WIP
- upward 'omni directional' camera SUPL
- terms BVREQ & BVACT replace BVCODE in toml
- brighter blue wheel mark
- reposition from wheel
- continual video rendering script
- failed 2nd attempt at a black background in world

File: genRobot.urdf (robot description, URDF)
Before this commit: robot test_robot, 7 links, 6 joints
Joints:
- joint base_to_fwheel: origin xyz=0.13 0 0.02 rpy=0 0 0 -> xyz=0.14 0 -0.011 rpy=0 0 0

Commit message: Checkpoint

File: genRobot.urdf (robot description, URDF)
Before this commit: robot test_robot, 7 links, 6 joints
Links:
- link base_link: mass 1 -> 4.54545454545454
- link fwheel: mass None -> 0; geometry collision cylinder length=0.005 radius=0.015; visual cylinder length=0.005 radius=0.015
- link lwheel: mass 0.1 -> 0.3; geometry collision cylinder length=0.02 radius=0.046; visual cylinder length=0.02 radius=0.046
- link lwheel_mark: mass None -> 0; geometry collision box size=0.01 0.022 0.08; visual box size=0.01 0.022 0.08
- link rwheel: mass 0.1 -> 0.3; geometry collision cylinder length=0.02 radius=0.046; visual cylinder length=0.02 radius=0.046
- link rwheel_mark: mass None -> 0; geometry collision box size=0.01 0.022 0.08; visual box size=0.01 0.022 0.08
Joints:
- joint base_to_fwheel: origin xyz=0.14 0 -0.011 rpy=0 0 0 -> xyz=0.14 0 0.010 rpy=0 0 0

Commit message: Checkpoint

File: genRobot.urdf (robot description, URDF)
Before this commit: robot test_robot, 7 links, 6 joints
Links:
- removed link base_link
- removed link fwheel_attach
- removed link lwheel_mark
- removed link rwheel_mark
- added link base, mass 10; collision box size=0.25 0.16 0.04; visual box size=0.25 0.16 0.04
- added link fattach; collision cylinder length=0.060 radius=0.023; visual cylinder length=0.060 radius=0.023
- added link lwheelmark, mass 0; collision box size=0.01 0.022 0.08; visual box size=0.01 0.022 0.08
- added link rwheelmark, mass 0; collision box size=0.01 0.022 0.08; visual box size=0.01 0.022 0.08
Joints:
- removed joint base_to_fattach
- removed joint base_to_fwheel
- removed joint base_to_lwheel
- removed joint base_to_rwheel
- removed joint lwheel_to_lwheel_mark
- removed joint rwheel_to_rwheel_mark
- added joint base_fattach: type fixed, parent base, child fattach, origin xyz=0 0 0 rpy=0 0 0
- added joint base_fwheel: type fixed, parent base, child fwheel, origin xyz=0.14 0 0.010 rpy=0 0 0
- added joint base_lwheel: type continuous, parent base, child lwheel, origin xyz=-0.05 0.115 0.046 rpy=0 0 -1.5707963, axis -1 0 0
- added joint base_rwheel: type continuous, parent base, child rwheel, origin xyz=-0.05 -0.115 0.046 rpy=0 0 1.5707963, axis 1 0 0
- added joint lwheel_lwheelmark: type fixed, parent lwheel, child lwheelmark, origin xyz=0 0 0 rpy=0 0 1.5707963
- added joint rwheel_rwheelmark: type fixed, parent rwheel, child rwheelmark, origin xyz=0 0 0 rpy=0 0 -1.5707963
